Commit message: XML description

File: urdf/spot.urdf (robot description, URDF)
Before this commit: robot spot, 16 links, 15 joints
Links:
- link body: mass None -> 16.25

File: urdf/spot.urdf.xacro (robot description, xacro)
@@ -5,10 +5,10 @@
         <visual>
             <geometry>
-                <mesh filename="~/Documents/PROJECTS-OF-MINE/spot_mujoco/urdf/meshes/body.dae" />
-            </geometry>
-        </visual>
-        <collision>
-            <geometry>
-                <mesh filename="~/Documents/PROJECTS-OF-MINE/spot_mujoco/urdf/meshes/body_collision.stl" />
+                <mesh filename="body.obj" />
+            </geometry>
+        </visual>
+        <collision>
+            <geometry>
+                <mesh filename="body_collision.stl" />
             </geometry>
         </collision>
@@ -43,10 +43,10 @@
         <visual>
             <geometry>
-                <mesh filename="~/Documents/PROJECTS-OF-MINE/spot_mujoco/urdf/meshes/front_left_hip.dae" />
-            </geometry>
-        </visual>
-        <collision>
-            <geometry>
-                <mesh filename="~/Documents/PROJECTS-OF-MINE/spot_mujoco/urdf/meshes/front_left_hip_collision.stl" />
+                <mesh filename="front_left_hip.obj" />
+            </geometry>
+        </visual>
+        <collision>
+            <geometry>
+                <mesh filename="front_left_hip_collision.stl" />
             </geometry>
         </collision>
@@ -78,10 +78,10 @@
         <visual>
             <geometry>
-                <mesh filename="~/Documents/PROJECTS-OF-MINE/spot_mujoco/urdf/meshes/front_left_upper_leg.dae" />
-            </geometry>
-        </visual>
-        <collision>
-            <geometry>
-                <mesh filename="~/Documents/PROJECTS-OF-MINE/spot_mujoco/urdf/meshes/front_left_upper_leg_collision.stl" />
+                <mesh filename="front_left_upper_leg.obj" />
+            </geometry>
+        </visual>
+        <collision>
+            <geometry>
+                <mesh filename="front_left_upper_leg_collision.stl" />
             </geometry>
         </collision>
@@ -113,10 +113,10 @@
         <visual>
             <geometry>
-                <mesh filename="~/Documents/PROJECTS-OF-MINE/spot_mujoco/urdf/meshes/front_left_lower_leg.dae" />
+                <mesh filename="front_left_lower_leg.obj" />
             </geometry>
         </visual>
         <collision name="front_left_lower_leg_fixed_joint_lump__front_bump_sensor">
             <geometry>
-                <mesh filename="~/Documents/PROJECTS-OF-MINE/spot_mujoco/urdf/meshes/front_left_lower_leg_collision.stl" />
+                <mesh filename="front_left_lower_leg_collision.stl" />
             </geometry>
         </collision>
@@ -161,10 +161,10 @@
         <visual>
             <geometry>
-                <mesh filename="~/Documents/PROJECTS-OF-MINE/spot_mujoco/urdf/meshes/front_right_hip.dae" />
-            </geometry>
-        </visual>
-        <collision>
-            <geometry>
-                <mesh filename="~/Documents/PROJECTS-OF-MINE/spot_mujoco/urdf/meshes/front_right_hip_collision.stl" />
+                <mesh filename="front_right_hip.obj" />
+            </geometry>
+        </visual>
+        <collision>
+            <geometry>
+                <mesh filename="front_right_hip_collision.stl" />
             </geometry>
         </collision>
@@ -196,10 +196,10 @@
         <visual>
             <geometry>
-                <mesh filename="~/Documents/PROJECTS-OF-MINE/spot_mujoco/urdf/meshes/front_right_upper_leg.dae" />
-            </geometry>
-        </visual>
-        <collision>
-            <geometry>
-                <mesh filename="~/Documents/PROJECTS-OF-MINE/spot_mujoco/urdf/meshes/front_right_upper_leg_collision.stl" />
+                <mesh filename="front_right_upper_leg.obj" />
+            </geometry>
+        </visual>
+        <collision>
+            <geometry>
+                <mesh filename="front_right_upper_leg_collision.stl" />
             </geometry>
         </collision>
@@ -231,10 +231,10 @@
         <visual>
             <geometry>
-                <mesh filename="~/Documents/PROJECTS-OF-MINE/spot_mujoco/urdf/meshes/front_right_lower_leg.dae" />
+                <mesh filename="front_right_lower_leg.obj" />
             </geometry>
         </visual>
         <collision name="front_right_lower_leg_fixed_joint_lump__front_bump_sensor">
             <geometry>
-                <mesh filename="~/Documents/PROJECTS-OF-MINE/spot_mujoco/urdf/meshes/front_right_lower_leg_collision.stl" />
+                <mesh filename="front_right_lower_leg_collision.stl" />
             </geometry>
         </collision>
@@ -279,10 +279,10 @@
         <visual>
             <geometry>
-                <mesh filename="~/Documents/PROJECTS-OF-MINE/spot_mujoco/urdf/meshes/rear_left_hip.dae" />
-            </geometry>
-        </visual>
-        <collision>
-            <geometry>
-                <mesh filename="~/Documents/PROJECTS-OF-MINE/spot_mujoco/urdf/meshes/rear_left_hip_collision.stl" />
+                <mesh filename="rear_left_hip.obj" />
+            </geometry>
+        </visual>
+        <collision>
+            <geometry>
+                <mesh filename="rear_left_hip_collision.stl" />
             </geometry>
         </collision>
@@ -314,10 +314,10 @@
         <visual>
             <geometry>
-                <mesh filename="~/Documents/PROJECTS-OF-MINE/spot_mujoco/urdf/meshes/rear_left_upper_leg.dae" />
-            </geometry>
-        </visual>
-        <collision>
-            <geometry>
-                <mesh filename="~/Documents/PROJECTS-OF-MINE/spot_mujoco/urdf/meshes/rear_left_upper_leg_collision.stl" />
+                <mesh filename="rear_left_upper_leg.obj" />
+            </geometry>
+        </visual>
+        <collision>
+            <geometry>
+                <mesh filename="rear_left_upper_leg_collision.stl" />
             </geometry>
         </collision>
@@ -349,10 +349,10 @@
         <visual>
             <geometry>
-                <mesh filename="~/Documents/PROJECTS-OF-MINE/spot_mujoco/urdf/meshes/rear_left_lower_leg.dae" />
+                <mesh filename="rear_left_lower_leg.obj" />
             </geometry>
         </visual>
         <collision name="rear_left_lower_leg_fixed_joint_lump__rear_bump_sensor">
             <geometry>
-                <mesh filename="~/Documents/PROJECTS-OF-MINE/spot_mujoco/urdf/meshes/rear_left_lower_leg_collision.stl" />
+                <mesh filename="rear_left_lower_leg_collision.stl" />
             </geometry>
         </collision>
@@ -397,10 +397,10 @@
         <visual>
             <geometry>
-                <mesh filename="~/Documents/PROJECTS-OF-MINE/spot_mujoco/urdf/meshes/rear_right_hip.dae" />
-            </geometry>
-        </visual>
-        <collision>
-            <geometry>
-                <mesh filename="~/Documents/PROJECTS-OF-MINE/spot_mujoco/urdf/meshes/rear_right_hip_collision.stl" />
+                <mesh filename="rear_right_hip.obj" />
+            </geometry>
+        </visual>
+        <collision>
+            <geometry>
+                <mesh filename="rear_right_hip_collision.stl" />
             </geometry>
         </collision>
@@ -432,10 +432,10 @@
         <visual>
             <geometry>
-                <mesh filename="~/Documents/PROJECTS-OF-MINE/spot_mujoco/urdf/meshes/rear_right_upper_leg.dae" />
-            </geometry>
-        </visual>
-        <collision>
-            <geometry>
-                <mesh filename="~/Documents/PROJECTS-OF-MINE/spot_mujoco/urdf/meshes/rear_right_upper_leg_collision.stl" />
+                <mesh filename="rear_right_upper_leg.obj" />
+            </geometry>
+        </visual>
+        <collision>
+            <geometry>
+                <mesh filename="rear_right_upper_leg_collision.stl" />
             </geometry>
         </collision>
@@ -467,10 +467,10 @@
         <visual>
             <geometry>
-                <mesh filename="~/Documents/PROJECTS-OF-MINE/spot_mujoco/urdf/meshes/rear_right_lower_leg.dae" />
+                <mesh filename="rear_right_lower_leg.obj" />
             </geometry>
         </visual>
         <collision name='rear_right_lower_leg_fixed_joint_lump__rear_bump_sensor'>
             <geometry>
-                <mesh filename="~/Documents/PROJECTS-OF-MINE/spot_mujoco/urdf/meshes/rear_right_lower_leg_collision.stl" />
+                <mesh filename="rear_right_lower_leg_collision.stl" />
             </geometry>
         </collision>
