Commit message: up

File: meshes/spot.urdf (robot description, URDF)
Before this commit: robot spot, 16 links, 15 joints
Links:
- link body: geometry collision mesh filename=body_collision.stl; visual mesh filename=body.dae
- link front_left_hip: geometry collision mesh filename=front_left_hip_collision.stl; visual mesh filename=front_left_hip.dae
- link front_left_lower_leg: geometry collision mesh filename=front_left_lower_leg_collision.stl; visual mesh filename=front_left_lower_leg.dae
- link front_left_upper_leg: geometry collision mesh filename=front_left_upper_leg_collision.stl; visual mesh filename=front_left_upper_leg.dae
- link front_right_hip: geometry collision mesh filename=front_right_hip_collision.stl; visual mesh filename=front_right_hip.dae
- link front_right_lower_leg: geometry collision mesh filename=front_right_lower_leg_collision.stl; visual mesh filename=front_right_lower_leg.dae
- link front_right_upper_leg: geometry collision mesh filename=front_right_upper_leg_collision.stl; visual mesh filename=front_right_upper_leg.dae
- link rear_left_hip: geometry collision mesh filename=rear_left_hip_collision.stl; visual mesh filename=rear_left_hip.dae
- link rear_left_lower_leg: geometry collision mesh filename=rear_left_lower_leg_collision.stl; visual mesh filename=rear_left_lower_leg.dae
- link rear_left_upper_leg: geometry collision mesh filename=rear_left_upper_leg_collision.stl; visual mesh filename=rear_left_upper_leg.dae
- link rear_right_hip: geometry collision mesh filename=rear_right_hip_collision.stl; visual mesh filename=rear_right_hip.dae
- link rear_right_lower_leg: geometry collision mesh filename=rear_right_lower_leg_collision.stl; visual mesh filename=rear_right_lower_leg.dae
- link rear_right_upper_leg: geometry collision mesh filename=rear_right_upper_leg_collision.stl; visual mesh filename=rear_right_upper_leg.dae
